File: Scematics/Printer-Related/HB-MOSFET.sch (KiCad schematic (older format))
At the start: 9 parts, among them P1 CONN_01X02, P2 CONN_01X02, P3 CONN_01X02, Q1 LOGIC, Q2 HI-POWER

Commit message: Random MOSFET Changes
Parts:
- gave numbers to parts that had none: 2
Connections:
- net at P2.1 (P1), Q2.1 (D): now also R3.1; no longer R3.2
- net at D1.2 (A): now also R3.2; no longer R3.1
- net +24V renamed +12V
Other:
- note added: "Heatbed-Anschluss\n"
- note added: "Schaltungs-MOSFET\nmit Heatsink"
- note added: "Status-LED\n(grün)"
- note added: "Steuer-Anschluss\n"
- note added: "Steuer-Logic\nNICHT-Gatter & Pullups"
- note added: "Stromanschluss\n"
- moved on the sheet: D1, P1, P2, P3, Q1, Q2, R1, R2, R3
